File: PCB/SubPCB.kicad_pcb (KiCad board)
At the start: 2 copper layers, 100 x 100 mm, 65 parts, among them U10 TLP222A, U11 TLP222A, U12 TLP222A, U13 TLP222A, U14 TLP222A, U15 TLP222A, U16 TLP222A, U17 TLP222A, U18 TLP222A, U2 TLP785, U3 TLP785, U38 MCP2562-E-P, U4 TLP785, U5 TLP785, U6 TLP785, U7 TLP785, U8 TLP785, U9 TLP785

Commit message: add
Parts:
- added J_CAN_TM1: Jump_3p, KAZAAAN:Conn_3pin, F.Cu at (20.3, 6.35)
- added R19: R_1608, Resistor_SMD:R_0603_1608Metric_Pad0.98x0.95mm_HandSolder, F.Cu at (16.5, 10.6)
- added RESET_SW: SW_Push, Button_Switch_THT:SW_PUSH_6mm_H5mm, F.Cu at (55.2, 20.6)
- added USER_SW: SW_Push, Button_Switch_THT:SW_PUSH_6mm_H5mm, F.Cu at (55.2, 32.1)
- moved Cir_Pwr_D 2.09 mm to (58.7, 14.6)
- moved R18 2.09 mm to (58.7, 10.8)
- renumbered D1 to Cir_Pwr_D
Connections:
- U_STM1 pad CN7_14: unconnected-(U_STM1A-CN7_RESET-PadCN7_14) -> Net-(U_STM1A-CN7_RESET)
- U_STM1 pad CN7_23: unconnected-(U_STM1A-PC13-PadCN7_23) -> Net-(U_STM1A-PC13)
Routing:
- net Net-(U_STM1A-PC13): track 0.00 -> 18.7 mm
- net Net-(U_STM1A-CN7_RESET): track 0.00 -> 15.6 mm
- net Net-(J_CAN1-Pin_3): track 9.65 -> 18.6 mm
- net Net-(J_CAN1-Pin_2): track 9.65 -> 16.8 mm
- net Net-(J_CAN_TM1-Pin_3): track 0.00 -> 3.83 mm
- net UART_TX: track 52.6 -> 55.6 mm
Other:
- board text added: "Open"
- board text added: "Term"
